Commit message: launch gazebo

File: bot00_description/install/bot00_description/share/bot00_description/urdf/urdf_intro.urdf (robot description, URDF)
Before this commit: robot bot00, 7 links, 6 joints
Links:
- link base_link: mass None -> 0.2; geometry collision cylinder length=0.12 radius=0.10; visual cylinder length=0.12 radius=0.10
- link caster_link: geometry collision sphere radius=0.016; visual sphere radius=0.016
- link imu_link: mass None -> 0.1; geometry collision box size=0.02 0.02 0.02; visual box size=0.02 0.02 0.02
- link laser_link: mass None -> 0.1; geometry collision cylinder length=0.02 radius=0.02; visual cylinder length=0.02 radius=0.02
- link left_wheel_link: mass None -> 0.2; geometry collision cylinder length=0.04 radius=0.032; visual cylinder length=0.04 radius=0.032
- link right_wheel_link: mass None -> 0.2; geometry collision cylinder length=0.04 radius=0.032; visual cylinder length=0.04 radius=0.032
